File: FloppyController.kicad_pcb (KiCad board)
At the start: 2 copper layers, 180 x 120 mm, 67 parts, among them J1 FDC2, J10 SEL2, J11 Spare, J12 CD1, J13 CD0, J14 FDC, J15 DOUT, J16 16MHz, J17 9.6MHz, J18 LED, J19 Data, J2 FDC1, J20 Addr, J21 Conn_01x13_Pin, J22 GND, J23 5V, J24 DS, J25 MOT1, J26 MOT2, J27 MOT4, J28 MOT3, J29 Conn_01x03_Pin, J3 FDC3, J4 FDC4, J5 DCH_EN, J6 Pin4, J7 Pin6, J8 Addr, J9 SEL1, U1 WD37C65, U10 74LS393, U3 HM6116, U4 74LS273, U5 28C256, U6 74LS138, U7 74LS04, U9 74LS04, Y1 16 MHz, Y2 9.6MHz

Commit message: Work in progress
Parts:
- U8: value ~ -> FDC9216
- Y1: value 16 MHz -> 9.6 MHz
- Y2: value 9.6MHz -> 16 MHz
- moved J11 92.9 mm to (69.7, 102.8)
- moved J22 27.2 mm to (126.0, 135.0)
- moved J13 24.0 mm to (150.0, 130.0)
- moved R7 22.7 mm to (56.1, 26.5), turned to 180 degrees
- moved J12 18.7 mm to (156.9, 130.0), turned to -90 degrees
- moved U4 15.1 mm to (39.5, 112.5)
- moved J21 11.9 mm to (59.4, 69.2)
- moved R6 11.7 mm to (47.8, 108.8), turned to 180 degrees
- moved R2 10.3 mm to (191.0, 127.0), turned to 180 degrees
- moved C3 10.3 mm to (46.2, 105.2), turned to 180 degrees
- moved R3 10.3 mm to (191.0, 131.0), turned to 180 degrees
- moved R4 10.3 mm to (191.0, 135.0), turned to 180 degrees
- moved U2 10.2 mm to (88.9, 53.1)
- moved R9 9.78 mm to (146.8, 64.7)
- moved R13 9.45 mm to (145.9, 93.1)
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Connections:
- J16 pad 1: /XT1 -> /XT2
- J16 pad 10: /1MHz -> /0.6MHz
- J16 pad 2: /16MHz -> /9.6MHz
- J16 pad 3: /XT1 -> /XT2
- J16 pad 4: /8MHz -> /4.8MHz
- J16 pad 5: /XT1 -> /XT2
- J16 pad 6: /4MHz -> /2.4MHz
- J16 pad 7: /XT1 -> /XT2
- J16 pad 8: /2MHz -> /1.2MHz
- J16 pad 9: /XT1 -> /XT2
- J17 pad 1: /XT2 -> /16MHz
- J17 pad 10: /0.6MHz -> /XT1
- J17 pad 2: /9.6MHz -> /XT1
- J17 pad 3: /XT2 -> /8MHz
- J17 pad 4: /4.8MHz -> /XT1
- J17 pad 5: /XT2 -> /4MHz
- J17 pad 6: /2.4MHz -> /XT1
- J17 pad 7: /XT2 -> /2MHz
- J17 pad 8: /1.2MHz -> /XT1
- J17 pad 9: /XT2 -> /1MHz
- J9 pad 3: Net-(J9-Pin_3) -> unconnected-(J9-Pin_3-Pad3)
- U10 pad 1: /16MHz -> /9.6MHz
- U10 pad 10: /2.4MHz -> /4MHz
- U10 pad 11: /4.8MHz -> /8MHz
- U10 pad 13: /9.6MHz -> /16MHz
- U10 pad 3: /8MHz -> /4.8MHz
- U10 pad 4: /4MHz -> /2.4MHz
- U10 pad 5: /2MHz -> /1.2MHz
- U10 pad 6: /1MHz -> /0.6MHz
- U10 pad 8: /0.6MHz -> /1MHz
- U10 pad 9: /1.2MHz -> /2MHz
- U7 pad 6: /16MHz -> /9.6MHz
- U7 pad 8: /9.6MHz -> /16MHz
- U9 pad 1: /A15 -> (no net)
- U9 pad 14: (no net) -> +5V
- U9 pad 2: Net-(J9-Pin_3) -> (no net)
- U9 pad 7: (no net) -> GND
Routing:
- net +5V: track 46.7 -> 432.5 mm
- net /A0: track 0.00 -> 235.2 mm, vias 0 -> 3
- net /D0: track 0.00 -> 170.5 mm, vias 0 -> 5
- net /D2: track 0.00 -> 169.8 mm, vias 0 -> 6
- net /D1: track 0.00 -> 168.7 mm, vias 0 -> 6
- net /A4: track 0.00 -> 142.5 mm, vias 0 -> 1
- net /A3: track 0.00 -> 140.8 mm, vias 0 -> 1
- net /A5: track 0.00 -> 136.7 mm, vias 0 -> 1
- net /A6: track 0.00 -> 136.1 mm, vias 0 -> 1
- net /A2: track 0.00 -> 129.0 mm, vias 0 -> 2
- net /A7: track 0.00 -> 128.8 mm, vias 0 -> 1
- net /A1: track 0.00 -> 124.5 mm, vias 0 -> 2
- net /RD: track 0.00 -> 121.3 mm, vias 0 -> 1
- net /A13: track 0.00 -> 115.4 mm, vias 0 -> 1
- net /WR: track 0.00 -> 111.4 mm, vias 0 -> 1
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