File: FloppyController.kicad_sch (KiCad schematic)
At the start: 26 parts, among them J1 Conn_02x17_Odd_Even, J2 Conn_02x17_Odd_Even, J3 Conn_02x17_Odd_Even, J4 Conn_02x17_Odd_Even, U4 74LS273

Commit message: Work in progress
Parts:
- added J10: SEL2, symbol Connector:Conn_01x03_Pin
- added J5: DCH_EN, Connector_PinHeader_2.54mm:PinHeader_1x02_P2.54mm_Vertical, symbol Connector:Conn_01x02_Pin
- added J6: Pin4, Connector_PinHeader_2.54mm:PinHeader_1x03_P2.54mm_Vertical, symbol Connector:Conn_01x03_Pin
- added J7: Pin6, symbol Connector:Conn_01x02_Pin
- added J8: Conn_02x08_Odd_Even, Connector_PinHeader_2.54mm:PinHeader_2x08_P2.54mm_Vertical, symbol Connector_Generic:Conn_02x08_Odd_Even
- added J9: SEL1, symbol Connector:Conn_01x03_Pin
- added U5: 28C256, symbol Memory_EEPROM:28C256
- added U6: 74LS138, symbol 74xx:74LS138
- added U7: 74LS04, symbol 74xx:74LS04
- C2, C4: value C -> 0.01
- C5: value C -> 0.1
- R6: value R -> 470
- R7: value R -> 1k
Connections:
- net +5V: now also C2.1, C3.1, C4.2, C5.1, C6.2, R6.1, R7.1, U2.40 (VCC), U2.42 (+5V), U3.24 (VCC), U4.20 (VCC), U5.28 (VCC), U6.16 (VCC)
- net DIR: now also U1.31 (-DIRC)
- net DSKCHG: now also U1.40 (-DCHG)
- net GND: now also C2.2, C3.2, C5.2, U2.20 (GND), U2.41 (GND2), U3.12 (GND), U4.10 (GND), J5.1 (Pin_1), U5.14 (GND), U6.8 (GND)
- net IDX: now also U1.43 (-IDX)
- net RDD: now also U1.21 (RDD)
- net STEP: now also U1.32 (-STEP)
- net TRK00: now also U1.42 (-TR00)
- net WR: now reaches U2.16 (P3.6)
- net WR: now also U3.21 (-WE)
- net RD: now reaches U2.17 (P3.7)
- net RD: now also U3.20 (-OE), U5.22 (~{OE})
- net A8: now reaches U2.21 (P2.0)
- net A8: now also U3.23 (A8), U5.25 (A8)
- net A9: now reaches U2.22 (P2.2)
- net A9: now also U3.22 (A9), U5.24 (A9)
- net A11: now reaches U2.24 (P2.3)
- net A11: now also U5.23 (A11), U6.1 (A0)
- net A12: now reaches U2.25 (P2.4)
- net A12: now also U5.2 (A12), U6.2 (A1)
- net A13: now reaches U2.26 (P2.5)
- net A13: now also U5.26 (A13), U6.3 (A2)
- net A14: now reaches U2.27 (P2.6)
- net A14: now also J10.1 (Pin_1), U5.1 (A14), U7.3
- net A15: now reaches U2.28 (P2.7)
- net A15: now also J9.1 (Pin_1), U7.1
- net PSEN: now reaches U2.29 (-PSEN)
- net PSEN: now also U5.20 (~{CS}), U6.6 (E3)
- net ALE: now reaches U2.30 (ALE)
- net ALE: now also U4.11 (Cp)
- net D7: now reaches U2.32 (P0.7)
- net D7: now also U1.14 (DB7), U3.17 (D7), U4.18 (D7), U5.19 (D7)
- net D6: now reaches U2.33 (P0.6)
- net D6: now also U1.13 (DB6), U3.16 (D6), U4.17 (D6), U5.18 (D6)
- net D5: now reaches U2.34 (P0.5)
- net D5: now also U1.12 (DB5), U3.15 (D5), U4.14 (D5), U5.17 (D5)
- net D4: now reaches U2.35 (P0.4)
- net D4: now also U1.11 (DB4), U3.14 (D4), U4.13 (D4), U5.16 (D4)
- net D3: now reaches U2.36 (P0.3)
- net D3: now also U1.10 (DB3), U3.13 (D3), U4.8 (D3), U5.15 (D3)
- net D2: now reaches U2.37 (P0.2)
- net D2: now also U1.9 (DB2), U3.11 (D2), U4.7 (D2), U5.13 (D2)
- net D1: now reaches U2.38 (P0.1)
- net D1: now also U1.8 (DB1), U3.10 (D1), U4.4 (D1), U5.12 (D1)
- net D0: now reaches U2.39 (P0.0)
- net D0: now also U1.7 (DB0), U3.9 (D0), U4.3 (D0), U5.11 (D0)
- net A7: now reaches U3.1 (A7)
- net A7: now also U4.19 (Q7), U5.3 (A7)
- net RAM: now reaches U3.18 (-CE)
- net RAM: now also J8.10 (Pin_10), J8.12 (Pin_12), J8.14 (Pin_14), J8.16 (Pin_16), J8.2 (Pin_2), J8.4 (Pin_4), J8.6 (Pin_6), J8.8 (Pin_8)
- net A10: now reaches U3.19 (A10)
- net A10: now also U2.22 (P2.2), U5.21 (A10)
- net A6: now reaches U3.2 (A6)
- net A6: now also U4.16 (Q6), U5.4 (A6)
- net A5: now reaches U3.3 (A5)
- net A5: now also U4.15 (Q5), U5.5 (A5)
- net A4: now reaches U3.4 (A4)
- net A4: now also U4.12 (Q4), U5.6 (A4)
- net A3: now reaches U3.5 (A3)
- net A3: now also U4.9 (Q3), U5.7 (A3)
- net A2: now reaches U3.6 (A2)
- net A2: now also U4.6 (Q2), U5.8 (A2)
- net A1: now reaches U3.7 (A1)
- net A1: now also U4.5 (Q1), U5.9 (A1)
- net A0: now reaches U3.8 (A0)
- net A0: now also U4.2 (Q0), U5.10 (A0)
- net at U4.1 (~{Mr}): now also R6.2
- net DCH: now reaches U1.17 (-DCHGEN)
- net DCH: now also J5.2 (Pin_2)
- net DS4: now reaches U1.37 (-DS4)
- net DS4: now also J7.1 (Pin_1)
- net HDL: now reaches U1.38 (-HDL)
- net HDL: now also J6.1 (Pin_1)
- net P4: now reaches J3.4 (Pin_4)
- net P4: now also J1.4 (Pin_4), J2.4 (Pin_4), J4.4 (Pin_4), J6.2 (Pin_2)
- net P6: now reaches J3.6 (Pin_6)
- net P6: now also J1.6 (Pin_6), J2.6 (Pin_6), J4.6 (Pin_6), J7.2 (Pin_2)
- net at R7.2: now also U5.27 (~{WE})
- new net: J8.1 (Pin_1), U6.15 (O0)
- new net: J8.11 (Pin_11), U6.10 (O5)
- new net: J8.13 (Pin_13), U6.9 (O6)
- new net: J8.15 (Pin_15), U6.7 (O7)
- new net: J8.3 (Pin_3), U6.14 (O1)
- new net: J8.5 (Pin_5), U6.13 (O2)
- new net: J8.7 (Pin_7), U6.12 (O3)
- new net: J8.9 (Pin_9), U6.11 (O4)
- new net: J9.3 (Pin_3), U7.2
- new net: J10.3 (Pin_3), U7.4
- new net SEL1: J9.2 (Pin_2), U6.4 (E1)
- new net SEL2: J10.2 (Pin_2), U6.5 (E2)
- new net USE: J6.3 (Pin_3)
Other:
- moved on the sheet: C2, C3, C4, C5, C6, R6, R7, U2, U3, U4

Commit message: Work in progress
Parts:
- added J11: Spare, symbol Connector:Conn_01x03_Pin
- added J12: CD1, symbol Connector:Conn_01x02_Pin
- added J13: CD0, symbol Connector:Conn_01x02_Pin
- added J14: FDC, symbol Connector:Conn_01x03_Pin
- added J15: Conn_01x04_Pin, Connector_PinHeader_2.54mm:PinHeader_1x04_P2.54mm_Vertical, symbol Connector:Conn_01x04_Pin
- added R11: 1k, symbol Device:R
- added R12, R13: R, symbol Device:R
- added U10: 74LS393, symbol 74xx:74LS393
- added unit 7 of U7
- added unit 3 of U7
- added unit 4 of U7
- added unit 6 of U7
- added unit 5 of U7
- added U8: ~, symbol Interface:FDC9216
- added U9: 74LS04, symbol 74xx:74LS04
- added Y1: 16 MHz, Crystal:Crystal_HC49-U_Vertical, symbol Device:Crystal
- added Y2: 9.6MHz, Crystal:Crystal_HC49-U_Vertical, symbol Device:Crystal
- C7, C8: value C -> 0.01
- J8: value Conn_02x08_Odd_Even -> Addr
- R10: value R -> 1k
- R8, R9: value R -> 470
- U1: value ~ -> WD37C65
Connections:
- net +5V: now also C7.1, C8.1, R10.1, R11.1, U10.14 (VCC), U7.14 (VCC)
- net A0: now also U1.4 (A0)
- net GND: now also C6.1, C7.2, C8.2, J12.2 (Pin_2), J13.2 (Pin_2), J15.1 (Pin_1), R12.2, R13.2, U10.7 (GND), U7.7 (GND), U8.4 (GND)
- net IDX: now also J15.4 (Pin_4)
- net RAM: no longer J8.10 (Pin_10), J8.12 (Pin_12), J8.14 (Pin_14), J8.16 (Pin_16), J8.6 (Pin_6), J8.8 (Pin_8)
- net RD: now also U1.1 (-RD)
- net RDD: now also J14.1 (Pin_1)
- net WDATA: now also U1.30 (-WD)
- net WGATE: now also U1.29 (-WE)
- net WR: now also U1.2 (-WR)
- net INT: now reaches U2.12 (P3.2)
- net INT: now also U1.16 (IRQ)
- net TC: now reaches U2.3 (P1.2)
- net TC: now also U1.6 (TC)
- net FDRST: now reaches U2.4 (P1.3)
- net FDRST: now also U1.20 (RST)
- net at R9.1: now also U7.13, Y2.1
- net at R9.2: now also U7.11, U7.12
- net at R8.1: now also U7.5, Y1.1
- net at R8.2: now also U7.6, U9.1
- net LDOR: now reaches U1.18 (-LDOR)
- net LDOR: now also J8.8 (Pin_8)
- net LDCR: now reaches U1.19 (-LDCR)
- net LDCR: now also J8.10 (Pin_10)
- net -XT2: now reaches U1.22 (-XT2)
- net XT2: now reaches U1.23 (XT2)
- net -XT1: now reaches U1.25 (-XT1)
- net XT1: now reaches U1.26 (XT1)
- net FDCS: now reaches U1.3 (-CS)
- net FDCS: now also J8.6 (Pin_6)
- net at R10.2: now also J13.1 (Pin_1), U8.5 (CD0)
- new net: J11.3 (Pin_3), J8.12 (Pin_12)
- new net: J11.2 (Pin_2), J8.14 (Pin_14)
- new net: J11.1 (Pin_1), J8.16 (Pin_16)
- new net: J14.2 (Pin_2), U8.1 (RDD)
- new net: R13.1, U10.12 (MR)
- new net: U9.2, U9.3, Y1.2
- new net: U7.10, U7.9, Y2.2
- new net: J12.1 (Pin_1), R11.2, U8.6 (CD1)
- new net: J15.2 (Pin_2), U8.7 (DOUT)
- new net: J15.3 (Pin_3), U8.2 (CLKOUT)
- new net: R12.1, U10.2 (MR)
- new net 0.6MHz: U10.8 (Q3)
- new net 1.2MHz: U10.9 (Q2)
- new net 16MHz: U10.1 (CP), U9.4
- new net 1MHz: U10.6 (Q3)
- new net 2.4MHz: U10.10 (Q1)
- new net 2MHz: U10.5 (Q2)
- new net 4.8MHz: U10.11 (Q0)
- new net 4MHz: U10.4 (Q1)
- new net 8MHz: U10.3 (Q0)
- new net 9.6MHz: U10.13 (CP), U7.8
Other:
- moved on the sheet: C7, C8, J8, R10, R6, R8, R9, U6

Commit message: Work in progress
Parts:
- added C9: 0.01, Capacitor_THT:C_Disc_D4.7mm_W2.5mm_P5.00mm, symbol Device:C
- added D1, D2: LED, LED_THT:LED_D5.0mm, symbol Device:LED
- added J16: 16MHz, Connector_PinHeader_2.54mm:PinHeader_2x05_P2.54mm_Vertical, symbol Connector_Generic:Conn_02x05_Odd_Even
- added J17: 9.6MHz, Connector_PinHeader_2.54mm:PinHeader_2x05_P2.54mm_Vertical, symbol Connector_Generic:Conn_02x05_Odd_Even
- added J18: LED, Connector_PinHeader_2.54mm:PinHeader_1x02_P2.54mm_Vertical, symbol Connector:Conn_01x02_Pin
- added J19: Data, Connector_PinSocket_2.54mm:PinSocket_1x09_P2.54mm_Vertical, symbol Connector:Conn_01x09_Pin
- added J20: Addr, Connector_PinHeader_2.54mm:PinHeader_1x17_P2.54mm_Vertical, symbol Connector:Conn_01x17_Pin
- added J21: Conn_01x13_Pin, Connector_PinHeader_2.54mm:PinHeader_1x13_P2.54mm_Vertical, symbol Connector:Conn_01x13_Pin
- added J22: GND, Connector_PinSocket_2.54mm:PinSocket_1x04_P2.54mm_Vertical, symbol Connector:Conn_01x04_Pin
- added J23: 5V, Connector_PinSocket_2.54mm:PinSocket_1x04_P2.54mm_Vertical, symbol Connector:Conn_01x04_Pin
- added J24: DS, Connector_PinHeader_2.54mm:PinHeader_1x04_P2.54mm_Vertical, symbol Connector:Conn_01x04_Pin
- added J25: MOT1, Connector_PinHeader_2.54mm:PinHeader_1x04_P2.54mm_Vertical, symbol Connector:Conn_01x04_Pin
- added J26: MOT2, Connector_PinHeader_2.54mm:PinHeader_1x04_P2.54mm_Vertical, symbol Connector:Conn_01x04_Pin
- added J27: MOT4, Connector_PinHeader_2.54mm:PinHeader_1x04_P2.54mm_Vertical, symbol Connector:Conn_01x04_Pin
- added J28: MOT3, Connector_PinHeader_2.54mm:PinHeader_1x04_P2.54mm_Vertical, symbol Connector:Conn_01x04_Pin
- added J29: Conn_01x03_Pin, Connector_PinHeader_2.54mm:PinHeader_1x03_P2.54mm_Vertical, symbol Connector:Conn_01x03_Pin
- added R14: 1k, Resistor_THT:R_Axial_DIN0207_L6.3mm_D2.5mm_P10.16mm_Horizontal, symbol Device:R
- added R15: R, Resistor_THT:R_Axial_DIN0207_L6.3mm_D2.5mm_P10.16mm_Horizontal, symbol Device:R
- C1, C2, C4, C5, C6, C7, C8: footprint (none) -> Capacitor_THT:C_Disc_D4.7mm_W2.5mm_P5.00mm
- C3: value C -> 0.01; footprint (none) -> Capacitor_THT:C_Disc_D4.7mm_W2.5mm_P5.00mm
- J1: value Conn_02x17_Odd_Even -> FDC2
- J10, J11, J14, J9: footprint (none) -> Connector_PinHeader_2.54mm:PinHeader_1x03_P2.54mm_Vertical
- J12, J13, J7: footprint (none) -> Connector_PinHeader_2.54mm:PinHeader_1x02_P2.54mm_Vertical
- J15: value Conn_01x04_Pin -> DOUT
- J2: value Conn_02x17_Odd_Even -> FDC1; footprint (none) -> Connector_PinHeader_2.54mm:PinHeader_2x17_P2.54mm_Vertical
- J3: value Conn_02x17_Odd_Even -> FDC3; footprint (none) -> Connector_PinHeader_2.54mm:PinHeader_2x17_P2.54mm_Vertical
- J4: value Conn_02x17_Odd_Even -> FDC4; footprint (none) -> Connector_PinHeader_2.54mm:PinHeader_2x17_P2.54mm_Vertical
- R1, R10, R11, R2, R3, R4, R5, R6, R7, R8, R9: footprint (none) -> Resistor_THT:R_Axial_DIN0207_L6.3mm_D2.5mm_P10.16mm_Horizontal
- R12, R13: value R -> 1k; footprint (none) -> Resistor_THT:R_Axial_DIN0207_L6.3mm_D2.5mm_P10.16mm_Horizontal
- U10, U7, U9: footprint (none) -> Package_DIP:DIP-14_W7.62mm_Socket_LongPads
- U2: footprint (none) -> Module:8051break
- U3: value ~ -> HM6116; footprint (none) -> Package_DIP:DIP-24_W15.24mm_Socket_LongPads
- U4: footprint (none) -> Package_DIP:DIP-20_W7.62mm_Socket_LongPads
- U5: footprint (none) -> Package_DIP:DIP-28_W15.24mm_Socket_LongPads
- U6: footprint (none) -> Package_DIP:DIP-16_W7.62mm_Socket_LongPads
- U8: value ~ -> FDC9216; footprint (none) -> Package_DIP:DIP-8_W7.62mm_Socket_LongPads
Connections:
- net +5V: now also U8.8 (VCC), C9.1, J23.1 (Pin_1), J23.2 (Pin_2), J23.3 (Pin_3), J23.4 (Pin_4), J29.3 (Pin_3)
- net 0.6MHz: now also J17.10 (Pin_10)
- net 1.2MHz: now also J17.8 (Pin_8)
- net 16MHz: now also U7.6, J16.2 (Pin_2); no longer U9.4
- net 1MHz: now also J16.10 (Pin_10)
- net 2.4MHz: now also J17.6 (Pin_6)
- net 2MHz: now also J16.8 (Pin_8)
- net 4.8MHz: now also J17.4 (Pin_4)
- net 4MHz: now also J16.6 (Pin_6)
- net 8MHz: now also J16.4 (Pin_4)
- net 9.6MHz: now also J17.2 (Pin_2)
- net A0: now also J20.2 (Pin_2)
- net A1: now also J20.3 (Pin_3)
- net A10: now also J20.12 (Pin_12)
- net A11: now also J20.13 (Pin_13)
- net A12: now also J20.14 (Pin_14)
- net A13: now also J20.15 (Pin_15)
- net A14: now also U9.3, J20.16 (Pin_16); no longer U7.3
- net A15: now also U9.1, J20.17 (Pin_17); no longer U7.1
- net A2: now also J20.4 (Pin_4)
- net A3: now also J20.5 (Pin_5)
- net A4: now also J20.6 (Pin_6)
- net A5: now also J20.7 (Pin_7)
- net A6: now also J20.8 (Pin_8)
- net A7: now also J20.9 (Pin_9)
- net A8: now also J20.10 (Pin_10)
- net A9: now also J20.11 (Pin_11)
- net D0: now also J19.9 (Pin_9)
- net D1: now also J19.8 (Pin_8)
- net D2: now also J19.7 (Pin_7)
- net D3: now also J19.6 (Pin_6)
- net D4: now also J19.5 (Pin_5)
- net D5: now also J19.4 (Pin_4)
- net D6: now also J19.3 (Pin_3)
- net D7: now also J19.2 (Pin_2)
- net DENSEL: now also J18.2 (Pin_2), R14.1
- net DRV1A: now also J25.2 (Pin_2)
- net DRV1B: now also J25.3 (Pin_3)
- net DRV2A: now also J26.2 (Pin_2)
- net DRV2B: now also J26.3 (Pin_3)
- net DRV3A: now also J28.2 (Pin_2)
- net DRV3B: now also J28.3 (Pin_3)
- net DRV4A: now also J27.2 (Pin_2)
- net DRV4B: now also J27.3 (Pin_3)
- net DS4: now also J24.4 (Pin_4)
- net GND: now also J15.4 (Pin_4), C9.2, D1.1 (K), D2.1 (K), J19.1 (Pin_1), J20.1 (Pin_1), J21.1 (Pin_1), J22.1 (Pin_1), J22.2 (Pin_2), J22.3 (Pin_3), J22.4 (Pin_4), J29.1 (Pin_1); no longer J15.1 (Pin_1)
- net HDSEL: now also U1.28 (-HS)
- net IDX: now also J15.1 (Pin_1); no longer J15.4 (Pin_4)
- net INT: now also J21.2 (Pin_2)
- net MOT1A: now also J25.4 (Pin_4)
- net MOT1B: now also J25.1 (Pin_1)
- net MOT2A: now also J26.4 (Pin_4)
- net MOT2B: now also J26.1 (Pin_1)
- net MOT3A: now also J28.4 (Pin_4)
- net MOT3B: now also J28.1 (Pin_1)
- net MOT4A: now also J27.4 (Pin_4)
- net MOT4B: now also J27.1 (Pin_1)
- net RD: now also J21.3 (Pin_3)
- net USE: now also J29.2 (Pin_2)
- net WPT: now also U1.41 (-WP)
- net WR: now also J21.4 (Pin_4)
- net XT1: now also J16.1 (Pin_1), J16.3 (Pin_3), J16.5 (Pin_5), J16.7 (Pin_7), J16.9 (Pin_9)
- net XT2: now also J17.1 (Pin_1), J17.3 (Pin_3), J17.5 (Pin_5), J17.7 (Pin_7), J17.9 (Pin_9)
- net P1.0: now reaches U2.1 (P1.0)
- net P1.0: now also J21.13 (Pin_13)
- net P3.0: now reaches U2.10 (P3.0)
- net P3.1: now reaches U2.11 (P3.1)
- net P3.3: now reaches U2.13 (P3.3)
- net P3.3: now also J21.7 (Pin_7)
- net P3.4: now reaches U2.14 (P3.4)
- net P3.4: now also J21.6 (Pin_6)
- net P3.5: now reaches U2.15 (P3.5)
- net P3.5: now also J21.5 (Pin_5)
- net P1.1: now reaches U2.2 (P1.1)
- net P1.1: now also J21.12 (Pin_12)
- net P1.4: now reaches U2.5 (P1.4)
- net P1.4: now also J21.11 (Pin_11)
- net P1.5: now reaches U2.6 (P1.5)
- net P1.5: now also J21.10 (Pin_10)
- net P1.6: now reaches U2.7 (P1.6)
- net P1.6: now also J21.9 (Pin_9)
- net P1.7: now reaches U2.8 (P1.7)
- net P1.7: now also J21.8 (Pin_8)
- net at J9.3 (Pin_3): now also U9.2; no longer U7.2
- net at R8.1, Y1.1: now also U7.1; no longer U7.5
- net at U7.4: now also U7.5, Y1.2; no longer J10.3 (Pin_3)
- net DS1: now reaches U1.33 (-DS1)
- net DS1: now also J24.1 (Pin_1)
- net DS2: now reaches U1.35 (-DS2)
- net DS2: now also J24.2 (Pin_2)
- net DS3: now reaches U1.36 (-DS3)
- net DS3: now also J24.3 (Pin_3)
- net RWC: now reaches U1.39 (-RWC)
- net RWC: now also J18.1 (Pin_1), R15.1
- new net: R8.2, U7.2, U7.3
- new net: D2.2 (A), R15.2
- new net: J10.3 (Pin_3), U9.4
- new net: D1.2 (A), R14.2
Other:
- moved on the sheet: C7, J15, U10C, U3, U7A, U7B, U7C, U7G, U9A, U9B

Commit message: Work in progress
Parts:
- Y1: value 16 MHz -> 9.6 MHz
- Y2: value 9.6MHz -> 16 MHz
Connections:
- net +5V: now also U9.14 (VCC)
- net 0.6MHz: now also J16.10 (Pin_10), U10.6 (Q3); no longer J17.10 (Pin_10), U10.8 (Q3)
- net 1.2MHz: now also J16.8 (Pin_8), U10.5 (Q2); no longer J17.8 (Pin_8), U10.9 (Q2)
- net 16MHz: now also J17.1 (Pin_1), U10.13 (CP), U7.8; no longer J16.2 (Pin_2), U10.1 (CP), U7.6
- net 1MHz: now also J17.9 (Pin_9), U10.8 (Q3); no longer J16.10 (Pin_10), U10.6 (Q3)
- net 2.4MHz: now also J16.6 (Pin_6), U10.4 (Q1); no longer J17.6 (Pin_6), U10.10 (Q1)
- net 2MHz: now also J17.7 (Pin_7), U10.9 (Q2); no longer J16.8 (Pin_8), U10.5 (Q2)
- net 4.8MHz: now also J16.4 (Pin_4), U10.3 (Q0); no longer J17.4 (Pin_4), U10.11 (Q0)
- net 4MHz: now also J17.5 (Pin_5), U10.10 (Q1); no longer J16.6 (Pin_6), U10.4 (Q1)
- net 8MHz: now also J17.3 (Pin_3), U10.11 (Q0); no longer J16.4 (Pin_4), U10.3 (Q0)
- net 9.6MHz: now also J16.2 (Pin_2), U10.1 (CP), U7.6; no longer J17.2 (Pin_2), U10.13 (CP), U7.8
- net A15: no longer U9.1
- net GND: now also U9.7 (GND)
- net XT1: now also J17.10 (Pin_10), J17.2 (Pin_2), J17.4 (Pin_4), J17.6 (Pin_6), J17.8 (Pin_8); no longer J16.1 (Pin_1), J16.3 (Pin_3), J16.5 (Pin_5), J16.7 (Pin_7), J16.9 (Pin_9)
- net XT2: now also J16.1 (Pin_1), J16.3 (Pin_3), J16.5 (Pin_5), J16.7 (Pin_7), J16.9 (Pin_9); no longer J17.1 (Pin_1), J17.3 (Pin_3), J17.5 (Pin_5), J17.7 (Pin_7), J17.9 (Pin_9)
- net at J9.3 (Pin_3): no longer U9.2
